Commit message: gripper changes

File: universal_robot/ur_description/urdf/ur5.urdf.xacro (robot description, xacro)
@@ -333,5 +333,5 @@
         <bodyName>vacuum_gripper</bodyName>
         <topicName>grasping</topicName>
-	<maxForce>50</maxForce>
+	<maxForce>1</maxForce>
         <maxDistance>0.05</maxDistance>
         <minDistance>0.01</minDistance>
@@ -368,5 +368,5 @@
         <bodyName>vacuum_gripper1</bodyName>
         <topicName>grasping1</topicName>
-	<maxForce>50</maxForce>
+	<maxForce>1</maxForce>
         <maxDistance>0.05</maxDistance>
         <minDistance>0.01</minDistance>
@@ -403,5 +403,5 @@
         <bodyName>vacuum_gripper2</bodyName>
         <topicName>grasping2</topicName>
-	<maxForce>50</maxForce>
+	<maxForce>1</maxForce>
         <maxDistance>0.05</maxDistance>
         <minDistance>0.01</minDistance>
@@ -438,5 +438,5 @@
         <bodyName>vacuum_gripper3</bodyName>
         <topicName>grasping2</topicName>
-	<maxForce>50</maxForce>
+	<maxForce>1</maxForce>
         <maxDistance>0.05</maxDistance>
         <minDistance>0.01</minDistance>
@@ -473,5 +473,5 @@
       <bodyName>vacuum_gripper4</bodyName>
       <topicName>grasping4</topicName>
-  <maxForce>50</maxForce>
+  <maxForce>1</maxForce>
       <maxDistance>0.05</maxDistance>
       <minDistance>0.01</minDistance>
@@ -508,5 +508,5 @@
       <bodyName>vacuum_gripper5</bodyName>
       <topicName>grasping5</topicName>
-<maxForce>50</maxForce>
+<maxForce>1</maxForce>
       <maxDistance>0.05</maxDistance>
       <minDistance>0.01</minDistance>
@@ -543,5 +543,5 @@
       <bodyName>vacuum_gripper6</bodyName>
       <topicName>grasping6</topicName>
-<maxForce>50</maxForce>
+<maxForce>1</maxForce>
       <maxDistance>0.05</maxDistance>
       <minDistance>0.01</minDistance>
@@ -578,5 +578,5 @@
       <bodyName>vacuum_gripper7</bodyName>
       <topicName>grasping7</topicName>
-<maxForce>50</maxForce>
+<maxForce>1</maxForce>
       <maxDistance>0.05</maxDistance>
       <minDistance>0.01</minDistance>
@@ -613,5 +613,5 @@
       <bodyName>vacuum_gripper8</bodyName>
       <topicName>grasping8</topicName>
-<maxForce>50</maxForce>
+<maxForce>1</maxForce>
       <maxDistance>0.05</maxDistance>
       <minDistance>0.01</minDistance>

File: ur5_ROS-Gazebo/urdf/red_box.urdf (robot description, URDF)
Before this commit: robot red_box, 1 links, 0 joints
Links:
- link base_link: mass 0.05 -> 0.005; geometry collision box size=0.2 0.2 0.2; visual box size=0.2 0.2 0.2
