Commit message: added bin

File: ur5_ROS-Gazebo/urdf/bin.urdf (robot description, URDF)
Before this commit: robot bin, 6 links, 5 joints
Links:
- link back: geometry collision box size=0.4 0.0001 0.4; visual box size=0.4 0.0001 0.4
- link bottom: geometry collision box size=0.4 0.6 0.0001; visual box size=0.4 0.6 0.0001
- link front: geometry collision box size=0.4 0.0001 0.4; visual box size=0.4 0.0001 0.4
- link left: geometry collision box size=0.0001 0.6 0.4; visual box size=0.0001 0.6 0.4
- link right: geometry collision box size=0.0001 0.6 0.4; visual box size=0.0001 0.6 0.4
